File: hardware/project_trace_kicad/Power.kicad_sch (KiCad schematic)
At the start: 8 parts, among them J1 FIT0587_Male, J2 FIT0587_Female, J3 Screw_Terminal_01x04, U1 UA78M33QDCYRQ1, U2 UA78M05QDCYRQ1

Commit message: Fix Mistakes, Reduce Scope, improve Flexibility
Parts:
- J1, J2: DigikeyPN (none) -> 1738-1437-ND
- J3: DigikeyPN (none) -> 732-691210910004-ND
- U1: DigikeyPN (none) -> 296-21208-1-ND
- U2: DigikeyPN (none) -> 296-19755-1-ND
Changed lines of the file:
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@@
+			)
+		)
+		(property "DigikeyPN" "296-21208-1-ND"
+			(at 191.77 87.63 0)
+			(effects
+				(font
+					(size 1.27 1.27)
+				)
+				(hide yes)
 			)
 		)
@@
 			)
 		)
+		(property "DigikeyPN" "1738-1437-ND"
+			(at 121.92 100.33 0)
+			(effects
+				(font
+					(size 1.27 1.27)
+				)
+				(hide yes)
+			)
+		)
 		(pin "1"
 		)
@@
 			)
 		)
+		(property "DigikeyPN" ""
+			(at 86.36 107.95 0)
+			(effects
+				(font
+					(size 1.27 1.27)
+				)
+				(hide yes)
+			)
+		)
 		(pin "1"
 		)
@@
 			)
 		)
+		(property "DigikeyPN" "1738-1437-ND"
+			(at 144.78 87.63 0)
+			(effects
+				(font
+					(size 1.27 1.27)
+				)
+				(hide yes)
+			)
+		)
 		(pin "1"
 		)
@@
 			)
 		)
+		(property "DigikeyPN" ""
+			(at 86.36 97.79 0)
+			(effects
+				(font
+					(size 1.27 1.27)
+				)
+				(hide yes)
+			)
+		)
 		(pin "1"
 		)
@@
 			)
 		)
+		(property "DigikeyPN" "732-691210910004-ND"
+			(at 152.4 90.17 0)
+			(effects
+				(font
+					(size 1.27 1.27)
+				)
+				(hide yes)
+			)
+		)
 		(pin "4"
 		)
@@
 			)
 		)
+		(property "DigikeyPN" "296-19755-1-ND"
+			(at 191.77 113.03 0)
+			(effects
+				(font
+					(size 1.27 1.27)
+				)
+				(hide yes)
+			)
+		)
 		(pin "3"
 		)
@@
 			(at 105.41 101.6 0)
 			(effects
+				(font
+					(size 1.27 1.27)
+				)
+				(hide yes)
+			)
+		)
+		(property "DigikeyPN" ""
+			(at 105.41 101.6 0)
+			(effects

Commit message: Before Changes to Input Section
Parts:
- A1: now not fitted
Changed lines of the file:
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@@
 		(in_bom yes)
 		(on_board no)
-		(dnp no)
+		(dnp yes)
 		(fields_autoplaced yes)
 		(property "Reference" "A1"

Commit message: Change designators, Improve Input Circuit
Parts:
- renumbered A1 to A501, BT1 to BT501, BT2 to BT502, J1 to J501, J2 to J502, J3 to J503, U1 to U501, U2 to U502
Changed lines of the file:
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@@
 	(wire
 		(pts
-			(xy 204.47 87.63) (xy 204.47 86.36)
-		)
-		(stroke
-			(width 0)
-			(type default)
-		)
-	)
-	(wire
-		(pts
-			(xy 199.39 87.63) (xy 204.47 87.63)
+			(xy 203.2 87.63) (xy 203.2 86.36)
+		)
+		(stroke
+			(width 0)
+			(type default)
+		)
+	)
+	(wire
+		(pts
+			(xy 199.39 87.63) (xy 203.2 87.63)
 		)
 		(stroke
@@
 	(wire
 		(pts
-			(xy 204.47 113.03) (xy 204.47 111.76)
+			(xy 203.2 113.03) (xy 203.2 111.76)
 		)
 		(stroke
@@
 	(wire
 		(pts
-			(xy 199.39 113.03) (xy 204.47 113.03)
+			(xy 199.39 113.03) (xy 203.2 113.03)
 		)
 		(stroke
@@
 		(dnp no)
 		(fields_autoplaced yes)
-		(property "Reference" "#PWR03"
+		(property "Reference" "#PWR0501"
 			(at 176.53 97.79 0)
 			(effects
@@
 			(project "project_trace_kicad"
 				(path "/af51f4e5-b952-4b0e-baf2-78a72fb86fcd/12a73351-c59a-4c39-a723-2f90ff2520c9"
-					(reference "#PWR03")
+					(reference "#PWR0501")
 					(unit 1)
 				)
@@
 		(on_board yes)
 		(dnp no)
-		(property "Reference" "#FLG02"
+		(property "Reference" "#FLG0502"
 			(at 167.64 93.345 0)
 			(effects
@@
 			(project "project_trace_kicad"
 				(path "/af51f4e5-b952-4b0e-baf2-78a72fb86fcd/12a73351-c59a-4c39-a723-2f90ff2520c9"
-					(reference "#FLG02")
+					(reference "#FLG0502")
 					(unit 1)
 				)
@@
 		(dnp no)
 		(fields_autoplaced yes)
-		(property "Reference" "U1"
+		(property "Reference" "U501"
 			(at 191.77 80.9455 0)
 			(effects
@@
 			(project "project_trace_kicad"
 				(path "/af51f4e5-b952-4b0e-baf2-78a72fb86fcd/12a73351-c59a-4c39-a723-2f90ff2520c9"
-					(reference "U1")
+					(reference "U501")
 					(unit 1)
 				)
@@
 		(dnp no)
 		(fields_autoplaced yes)
-		(property "Reference" "J1"
+		(property "Reference" "J501"
 			(at 122.6312 100.3878 0)
 			(effects
@@
 			(project "project_trace_kicad"
 				(path "/af51f4e5-b952-4b0e-baf2-78a72fb86fcd/12a73351-c59a-4c39-a723-2f90ff2520c9"
-					(reference "J1")
+					(reference "J501")
 					(unit 1)
 				)
@@
 		(dnp no)
 		(fields_autoplaced yes)
-		(property "Reference" "BT2"
+		(property "Reference" "BT502"
 			(at 83.439 104.8963 0)
 			(effects
@@
 			(project "project_trace_kicad"
 				(path "/af51f4e5-b952-4b0e-baf2-78a72fb86fcd/12a73351-c59a-4c39-a723-2f90ff2520c9"
-					(reference "BT2")
+					(reference "BT502")
 					(unit 1)
 				)
@@
 		(on_board no)
 		(dnp no)
-		(property "Reference" "J2"
+		(property "Reference" "J502"
 			(at 136.906 87.4917 0)
 			(do_not_autoplace yes)
@@
 			(project "project_trace_kicad"
 				(path "/af51f4e5-b952-4b0e-baf2-78a72fb86fcd/12a73351-c59a-4c39-a723-2f90ff2520c9"
-					(reference "J2")
+					(reference "J502")
 					(unit 1)
 				)
@@
 	(symbol
 		(lib_id "power:+3V3")
-		(at 204.47 86.36 0)
+		(at 203.2 86.36 0)
 		(unit 1)
 		(exclude_from_sim no)
@@
 		(dnp no)
 		(fields_autoplaced yes)
-		(property "Reference" "#PWR04"
-			(at 204.47 90.17 0)
+		(property "Reference" "#PWR0504"
+			(at 203.2 90.17 0)
 			(effects
 				(font
@@
 		)
 		(property "Value" "+3V3"
-			(at 204.47 82.2269 0)
+			(at 203.2 82.2269 0)
 			(effects
 				(font
@@
 		)
 		(property "Footprint" ""
-			(at 204.47 86.36 0)
+			(at 203.2 86.36 0)
 			(effects
 				(font
@@
 		)
 		(property "Datasheet" ""
-			(at 204.47 86.36 0)
+			(at 203.2 86.36 0)
 			(effects
 				(font
@@
 		)
 		(property "Description" "Power symbol creates a global label with name \"+3V3\""
-			(at 204.47 86.36 0)
+			(at 203.2 86.36 0)
 			(effects
 				(font
@@
 			(project "project_trace_kicad"
 				(path "/af51f4e5-b952-4b0e-baf2-78a72fb86fcd/12a73351-c59a-4c39-a723-2f90ff2520c9"
-					(reference "#PWR04")
+					(reference "#PWR0504")
 					(unit 1)
 				)
@@
 		(dnp no)
 		(fields_autoplaced yes)
-		(property "Reference" "BT1"
+		(property "Reference" "BT501"
 			(at 83.439 94.7363 0)
 			(effects
@@
 			(project "project_trace_kicad"
 				(path "/af51f4e5-b952-4b0e-baf2-78a72fb86fcd/12a73351-c59a-4c39-a723-2f90ff2520c9"
-					(reference "BT1")
+					(reference "BT501")
 					(unit 1)
 				)
@@
 		(on_board yes)
 		(dnp no)
-		(property "Reference" "J3"
+		(property "Reference" "J503"
 			(at 150.368 91.44 0)
 			(effects
@@
 			(project "project_trace_kicad"
 				(path "/af51f4e5-b952-4b0e-baf2-78a72fb86fcd/12a73351-c59a-4c39-a723-2f90ff2520c9"
-					(reference "J3")
+					(reference "J503")
 					(unit 1)
 				)
@@
 		(dnp no)
 		(fields_autoplaced yes)
-		(property "Reference" "U2"
+		(property "Reference" "U502"
 			(at 191.77 106.3455 0)
 			(effects
@@
 			(project "project_trace_kicad"
 				(path "/af51f4e5-b952-4b0e-baf2-78a72fb86fcd/12a73351-c59a-4c39-a723-2f90ff2520c9"
-					(reference "U2")
+					(reference "U502")
 					(unit 1)
 				)
@@
 		(dnp yes)
 		(fields_autoplaced yes)
-		(property "Reference" "A1"
+		(property "Reference" "A501"
 			(at 105.41 92.5025 0)
 			(effects
@@
 			(project "project_trace_kicad"
 				(path "/af51f4e5-b952-4b0e-baf2-78a72fb86fcd/12a73351-c59a-4c39-a723-2f90ff2520c9"
-					(reference "A1")
+					(reference "A501")
 					(unit 1)
 				)
@@
 	(symbol
 		(lib_id "power:+5V")
-		(at 204.47 111.76 0)
+		(at 203.2 111.76 0)
 		(unit 1)
 		(exclude_from_sim no)
@@
 		(dnp no)
 		(fields_autoplaced yes)
-		(property "Reference" "#PWR05"
-			(at 204.47 115.57 0)
+		(property "Reference" "#PWR0505"
+			(at 203.2 115.57 0)
 			(effects
 				(font
@@
 		)
 		(property "Value" "+5V"
-			(at 204.47 107.6269 0)
+			(at 203.2 107.6269 0)
 			(effects
 				(font
@@
 		)
 		(property "Footprint" ""
-			(at 204.47 111.76 0)
+			(at 203.2 111.76 0)
 			(effects
 				(font
@@
 		)
 		(property "Datasheet" ""
-			(at 204.47 111.76 0)
+			(at 203.2 111.76 0)
 			(effects
 				(font
@@
 		)
 		(property "Description" "Power symbol creates a global label with name \"+5V\""
-			(at 204.47 111.76 0)
+			(at 203.2 111.76 0)
 			(effects
 				(font
@@
 			(project "project_trace_kicad"
 				(path "/af51f4e5-b952-4b0e-baf2-78a72fb86fcd/12a73351-c59a-4c39-a723-2f90ff2520c9"
-					(reference "#PWR05")
+					(reference "#PWR0505")
 					(unit 1)
 				)
@@
 		(dnp no)
 		(fields_autoplaced yes)
-		(property "Reference" "#PWR02"
+		(property "Reference" "#PWR0503"
 			(at 191.77 128.27 0)
 			(effects
@@
 			(project "project_trace_kicad"
 				(path "/af51f4e5-b952-4b0e-baf2-78a72fb86fcd/12a73351-c59a-4c39-a723-2f90ff2520c9"
-					(reference "#PWR02")
+					(reference "#PWR0503")
 					(unit 1)
 				)
@@
 		(dnp no)
 		(fields_autoplaced yes)
-		(property "Reference" "#FLG01"
+		(property "Reference" "#FLG0501"
 			(at 167.64 84.455 0)
 			(effects
@@
 			(project "project_trace_kicad"
 				(path "/af51f4e5-b952-4b0e-baf2-78a72fb86fcd/12a73351-c59a-4c39-a723-2f90ff2520c9"
-					(reference "#FLG01")
+					(reference "#FLG0501")
 					(unit 1)
 				)
@@
 		(dnp no)
 		(fields_autoplaced yes)
-		(property "Reference" "#PWR01"
+		(property "Reference" "#PWR0502"
 			(at 191.77 102.87 0)
 			(effects
@@
 			(project "project_trace_kicad"
 				(path "/af51f4e5-b952-4b0e-baf2-78a72fb86fcd/12a73351-c59a-4c39-a723-2f90ff2520c9"
-					(reference "#PWR01")
+					(reference "#PWR0502")
 					(unit 1)
 				)

Commit message: Improve Inputs, Source Parts, Add Credits
Parts:
- A501, BT501, BT502: DigikeyPN (none) -> N/A
Other:
- company: Alexander Nybo Olsen -> (none)
- title: Power -> Multilloscope - Power
Changed lines of the file:
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@@
 	(paper "A4")
 	(title_block
-		(title "Power")
+		(title "Multilloscope - Power")
 		(date "2026-03-19")
 		(rev "1")
-		(company "Alexander Nybo Olsen")
+		(comment 1 "Laurits K. Hillemann")
+		(comment 2 "Alexander N. Olsen")
 	)
 	(junction
@@
 			)
 		)
-		(property "DigikeyPN" ""
+		(property "DigikeyPN" "N/A"
 			(at 86.36 107.95 0)
 			(effects
@@
 			)
 		)
-		(property "DigikeyPN" ""
+		(property "DigikeyPN" "N/A"
 			(at 86.36 97.79 0)
 			(effects
@@
 			)
 		)
-		(property "DigikeyPN" ""
+		(property "DigikeyPN" "N/A"
 			(at 105.41 101.6 0)
 			(effects

Commit message: Lotsa Changes
Parts:
- J502: now not fitted
Connections:
- no-connect marks 0 -> 2

Commit message: Work on PCB, Fix bugs, Improve noise performance
Parts:
- added C501, C502, C503, C504: 100u, Capacitor_THT:CP_Radial_D6.3mm_P2.50mm, symbol Device:C_Polarized
- J502: now fitted
Connections:
- net +3V3: now also C501.1
- net +5V: now also C502.1
- net GND: now also C501.2, C502.2, C503.2, C504.2
- net at J503.1 (Pin_1), J503.3 (Pin_3), U501.1 (IN)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: now also C503.1, C504.1
Other:
- moved on the sheet: U501, U502

Commit message: Address Review Comments
Parts:
- removed C501, C502: 100u, Capacitor_THT:CP_Radial_D6.3mm_P2.50mm, symbol Device:C_Polarized
- added C401, C402: 10u, Capacitor_THT:CP_Radial_D6.3mm_P2.50mm, symbol Device:C_Polarized
- C503, C504: value 100u -> 47u
Connections:
- net +3V3: now also C401.1
- net +5V: now also C402.1
- net GND: now also C401.2, C402.2
- net VBAT: now reaches C503.1, C504.1, J503.1 (Pin_1), J503.3 (Pin_3), U501.1 (IN), U502.1 (IN)

Commit message: UI updated, CLK implemented, Parts labeled as Donotplace in power
Parts:
- BT501, BT502, J501: now not fitted
Changed lines of the file:
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@@
 	(title_block
 		(title "Multilloscope - Power")
-		(date "2026-03-19")
+		(date "2026-04-06")
 		(rev "1")
 		(comment 1 "Laurits K. Hillemann")
@@
 		(on_board no)
 		(in_pos_files yes)
-		(dnp no)
+		(dnp yes)
 		(fields_autoplaced yes)
 		(property "Reference" "J501"
@@
 		(on_board no)
 		(in_pos_files yes)
-		(dnp no)
+		(dnp yes)
 		(fields_autoplaced yes)
 		(property "Reference" "BT502"
@@
 		(on_board no)
 		(in_pos_files yes)
-		(dnp no)
+		(dnp yes)
 		(fields_autoplaced yes)
 		(property "Reference" "BT501"
