File: hardware/project_trace_kicad/project_trace_kicad.kicad_pcb (KiCad board)
At the start: 4 copper layers, 100 x 100 mm, 101 parts, among them J204 Screw_Terminal_01x04, J205 Conn_Coaxial, J503 Screw_Terminal_01x04, U201 TLE2426xLP, U202 AQW280SX, U203 AQW282SX, U204 OPA2837IRUNT, U205 TS5A23159DGS, U206 OPA2837IRUNT, U301 THS4131IDR, U303 ADS1602, U304 MCP6499T, U305 LM4040DBZ-2.5, U306 LM4040DBZ-4.1, U501 UA78M33QDCYRQ1, U502 UA78M05QDCYRQ1, U503 NUCLEO-H753ZI

Commit message: Address Review Comments
Parts:
- added C213: 100n, Capacitor_SMD:C_0603_1608Metric_Pad1.08x0.95mm_HandSolder, F.Cu at (88.7, 121.5)
- added C401: 10u, Capacitor_THT:CP_Radial_D6.3mm_P2.50mm, F.Cu at (75.4, 105.1)
- added C402: 10u, Capacitor_THT:CP_Radial_D6.3mm_P2.50mm, F.Cu at (75.4, 113.0)
- added R310: 47k, Resistor_THT:R_Axial_DIN0207_L6.3mm_D2.5mm_P10.16mm_Horizontal, F.Cu at (84.2, 103.2)
- added TP302: TestPoint, TestPoint:TestPoint_Pad_1.5x1.5mm, F.Cu at (84.4, 107.0)
- added TP303: TestPoint, TestPoint:TestPoint_Pad_1.5x1.5mm, F.Cu at (84.4, 110.6)
- added TP304: TestPoint, TestPoint:TestPoint_Pad_1.5x1.5mm, F.Cu at (84.4, 114.1)
- added U207: SN74LVC2G14DBV, Package_TO_SOT_SMD:SOT-23-6_Handsoldering, F.Cu at (85.5, 120.3)
- C503, C504: value 100u -> 47u
- moved JP205 0.95 mm to (134.9, 121.5), turned to 0 degrees
Routing:
- net Net-(JP204-B): track 16.7 -> 17.8 mm
- net Net-(JP205-A): track 7.85 -> 7.32 mm
- net GND: vias 85 -> 84

Commit message: Before using stashed changes
Parts:
- added C303: 100n, Capacitor_SMD:C_0603_1608Metric_Pad1.08x0.95mm_HandSolder, B.Cu at (162.8, 139.0)
- added C328: 47u, Capacitor_THT:CP_Radial_D6.3mm_P2.50mm, F.Cu at (157.7, 118.1)
- added C329: 47u, Capacitor_THT:CP_Radial_D6.3mm_P2.50mm, F.Cu at (157.7, 125.2)
- added J602: Conn_01x14_Socket, ProjectTraceFootprints:JST_BM14B-GHS-TBT_LF__SN__N_, F.Cu at (242.2, 113.3)
- added JP303: SolderJumper_2_Open, Jumper:SolderJumper-2_P1.3mm_Open_RoundedPad1.0x1.5mm, B.Cu at (159.5, 143.2)
- added RV301: 10k, Potentiometer_THT:Potentiometer_Bourns_3266W_Vertical, F.Cu at (160.5, 154.4)
- added RV302: 10k, Potentiometer_THT:Potentiometer_Bourns_3266W_Vertical, F.Cu at (160.5, 160.4)
- added RV303: 10k, Potentiometer_THT:Potentiometer_Bourns_3266W_Vertical, F.Cu at (160.5, 166.5)
- added U302: ~, ProjectTraceFootprints:IC_625L3C040M00000_CTS-M, B.Cu at (162.9, 141.7)
- moved U207 19.3 mm to (66.5, 124.0)
- moved C213 19.3 mm to (69.7, 125.1)
- moved C321 1.12 mm to (154.9, 144.1), turned to 180 degrees
Connections:
- net Net-(J503-Pin_1) renamed VBAT
- C322 pad 2: +3V3 -> unconnected-(C322-Pad2)
- U303 pad 40: /ADC/CLK -> Net-(JP303-B)
- U303 pad 41: GND -> unconnected-(U303C-AGND-Pad41)
- U306 pad 1: Net-(U304C-+) -> unconnected-(U306-K-Pad1)
- U503 pad 8_4: /ADC/CLK -> unconnected-(U503C-PC9-Pad8_4)
Routing:
- net Net-(JP303-B): track 0.00 -> 10.8 mm, vias 0 -> 1
- net +5V: track 55.9 -> 58.5 mm, vias 8 -> 9
- net +3V3: track 38.8 -> 40.3 mm
- net GND: vias 84 -> 86
